File: SNES_USB_C_power.kicad_sch (KiCad schematic)
At the start: 24 parts, among them J1 USB4125-GF-A-0190, J2 Conn_01x02_Pin, Q1 AON6414A, Q2 AON6414A, SW1 SW_DIP_x03, U1 AP33771

Commit message: Update title and revision in schematic
Other:
- title: (none) -> Configurable USB C PD Decoy
Changed lines of the file:
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@@
 	(generator_version "8.0")
 	(paper "A4")
+	(title_block
+		(title "Configurable USB C PD Decoy")
+		(date "2024-06-03")
+		(rev "A")
+	)
 	(junction
 		(at 113.03 88.9)
